File: hw/led_bulb.kicad_pcb (KiCad board)
At the start: 2 copper layers, 92.4 x 91.4 mm, 170 parts, among them P1 USB_OTG, P10 CONN_01X02, P11 CONN_01X02, P12 CONN_01X02, P13 CONN_01X02, P14 CONN_01X02, P15 CONN_01X02, P16 CONN_01X02, P17 CONN_01X02, P18 CONN_01X02, P19 CONN_01X02, P2 CONN_01X02, P20 CONN_01X02, P21 CONN_01X02, P22 CONN_01X02, P23 CONN_01X02, P24 CONN_01X02, P25 CONN_01X02, P26 CONN_01X02, P27 CONN_01X02, P28 CONN_01X02, P29 CONN_01X02, P3 CONN_01X02, P30 CONN_01X02, P31 CONN_01X02, P32 CONN_01X02, P33 CONN_01X02, P4 CONN_01X02, P5 CONN_01X02, P6 CONN_01X02, P7 CONN_01X02, P8 CONN_01X02, P9 CONN_01X02, Q1 Q_NPN_EBC, Q2 Q_NPN_EBC, SW1 RST, SW2 FLASH, U1 CP2102, U3 ESP-12E, U4 AP1117D33

Commit message: Started work on v4.1 of hardware
Parts:
- Q1, Q2: value Q_NPN_EBC -> S8050
- U1: value CP2102 -> CP2102-GM
Connections:
- net Net-(LED43-Pad4) renamed Vv_USB
- LED13 pad 3: Net-(LED13-Pad3) -> GND
- LED13 pad 4: Net-(LED13-Pad4) -> V_USB
- LED14 pad 3: Net-(LED14-Pad3) -> GND
- LED14 pad 4: Net-(LED14-Pad4) -> V_USB
- LED15 pad 3: Net-(LED15-Pad3) -> GND
- LED15 pad 4: Net-(LED15-Pad4) -> V_USB
- LED16 pad 3: Net-(LED16-Pad3) -> GND
- LED16 pad 4: Net-(LED16-Pad4) -> V_USB
- LED17 pad 3: Net-(LED13-Pad3) -> GND
- LED17 pad 4: Net-(LED13-Pad4) -> V_USB
- LED18 pad 3: Net-(LED14-Pad3) -> GND
- LED18 pad 4: Net-(LED14-Pad4) -> V_USB
- LED19 pad 3: Net-(LED15-Pad3) -> GND
- LED19 pad 4: Net-(LED15-Pad4) -> V_USB
- LED20 pad 3: Net-(LED16-Pad3) -> GND
- LED20 pad 4: Net-(LED16-Pad4) -> V_USB
- LED21 pad 3: Net-(LED13-Pad3) -> GND
- LED21 pad 4: Net-(LED13-Pad4) -> V_USB
- LED22 pad 3: Net-(LED14-Pad3) -> GND
- LED22 pad 4: Net-(LED14-Pad4) -> V_USB
- LED23 pad 3: Net-(LED15-Pad3) -> GND
- LED23 pad 4: Net-(LED15-Pad4) -> V_USB
- LED24 pad 3: Net-(LED16-Pad3) -> GND
- LED24 pad 4: Net-(LED16-Pad4) -> V_USB
- LED25 pad 3: Net-(LED13-Pad3) -> GND
- LED25 pad 4: Net-(LED13-Pad4) -> V_USB
- LED26 pad 3: Net-(LED14-Pad3) -> GND
- LED26 pad 4: Net-(LED14-Pad4) -> V_USB
- LED27 pad 3: Net-(LED15-Pad3) -> GND
- LED27 pad 4: Net-(LED15-Pad4) -> V_USB
- LED28 pad 3: Net-(LED16-Pad3) -> GND
- LED28 pad 4: Net-(LED16-Pad4) -> V_USB
- LED29 pad 3: Net-(LED13-Pad3) -> GND
- LED29 pad 4: Net-(LED13-Pad4) -> V_USB
- LED30 pad 3: Net-(LED14-Pad3) -> GND
- LED30 pad 4: Net-(LED14-Pad4) -> V_USB
- LED31 pad 3: Net-(LED15-Pad3) -> GND
- LED31 pad 4: Net-(LED15-Pad4) -> V_USB
- LED32 pad 3: Net-(LED16-Pad3) -> GND
- LED32 pad 4: Net-(LED16-Pad4) -> V_USB
- LED33 pad 3: Net-(LED13-Pad3) -> GND
- LED33 pad 4: Net-(LED13-Pad4) -> V_USB
- LED34 pad 3: Net-(LED14-Pad3) -> GND
- LED34 pad 4: Net-(LED14-Pad4) -> V_USB
- LED35 pad 3: Net-(LED15-Pad3) -> GND
- LED35 pad 4: Net-(LED15-Pad4) -> V_USB
- LED36 pad 3: Net-(LED16-Pad3) -> GND
- LED36 pad 4: Net-(LED16-Pad4) -> V_USB
- LED37 pad 3: Net-(LED13-Pad3) -> GND
- LED37 pad 4: Net-(LED13-Pad4) -> V_USB
- LED38 pad 3: Net-(LED14-Pad3) -> GND
- LED38 pad 4: Net-(LED14-Pad4) -> V_USB
- LED39 pad 3: Net-(LED15-Pad3) -> GND
- LED39 pad 4: Net-(LED15-Pad4) -> V_USB
- LED40 pad 3: Net-(LED16-Pad3) -> GND
- LED40 pad 4: Net-(LED16-Pad4) -> V_USB
- LED41 pad 3: Net-(LED41-Pad3) -> GND
- LED41 pad 4: Net-(LED41-Pad4) -> V_USB
- LED42 pad 3: Net-(LED42-Pad3) -> GND
- LED42 pad 4: Net-(LED42-Pad4) -> V_USB
- LED43 pad 3: Net-(LED43-Pad3) -> GND
- LED44 pad 3: Net-(LED44-Pad3) -> GND
- LED44 pad 4: Net-(LED44-Pad4) -> V_USB
- LED45 pad 3: Net-(LED42-Pad3) -> GND
- LED45 pad 4: Net-(LED42-Pad4) -> V_USB
- LED46 pad 3: Net-(LED41-Pad3) -> GND
- LED46 pad 4: Net-(LED41-Pad4) -> V_USB
- LED47 pad 3: Net-(LED43-Pad3) -> GND
- LED48 pad 3: Net-(LED44-Pad3) -> GND
- LED48 pad 4: Net-(LED44-Pad4) -> V_USB
- LED49 pad 3: Net-(LED42-Pad3) -> GND
- LED49 pad 4: Net-(LED42-Pad4) -> V_USB
- LED50 pad 3: Net-(LED41-Pad3) -> GND
- LED50 pad 4: Net-(LED41-Pad4) -> V_USB
- LED51 pad 3: Net-(LED43-Pad3) -> GND
- LED52 pad 3: Net-(LED44-Pad3) -> GND
- LED52 pad 4: Net-(LED44-Pad4) -> V_USB
- LED53 pad 3: Net-(LED41-Pad3) -> GND
- LED53 pad 4: Net-(LED41-Pad4) -> V_USB
- P11 pad 1: Net-(LED13-Pad3) -> GND
- P11 pad 2: Net-(LED13-Pad4) -> V_USB
- P13 pad 1: Net-(LED14-Pad3) -> GND
- P13 pad 2: Net-(LED14-Pad4) -> V_USB
- P15 pad 1: Net-(LED15-Pad3) -> GND
- P15 pad 2: Net-(LED15-Pad4) -> V_USB
- P17 pad 1: Net-(LED16-Pad3) -> GND
- P17 pad 2: Net-(LED16-Pad4) -> V_USB
- P19 pad 1: Net-(LED41-Pad3) -> GND
- P19 pad 2: Net-(LED41-Pad4) -> V_USB
- P21 pad 1: Net-(LED42-Pad3) -> GND
- P21 pad 2: Net-(LED42-Pad4) -> V_USB
- P23 pad 1: Net-(LED43-Pad3) -> GND
- P25 pad 1: Net-(LED44-Pad3) -> GND
- P25 pad 2: Net-(LED44-Pad4) -> V_USB
- P27 pad 1: Net-(LED13-Pad4) -> V_USB
- P27 pad 2: Net-(LED13-Pad3) -> GND
- P29 pad 1: Net-(LED14-Pad4) -> V_USB
- P29 pad 2: Net-(LED14-Pad3) -> GND
- P31 pad 1: Net-(LED15-Pad4) -> V_USB
- P31 pad 2: Net-(LED15-Pad3) -> GND
- P33 pad 1: Net-(LED16-Pad4) -> V_USB
- P33 pad 2: Net-(LED16-Pad3) -> GND
- Q1 pad 1: DTR -> Net-(Q1-Pad1)
- Q1 pad 2: Net-(Q1-Pad2) -> DTR
- Q2 pad 1: RTS -> Net-(Q2-Pad1)
- Q2 pad 2: Net-(Q2-Pad2) -> RTS
- R6 pad 2: Net-(Q1-Pad2) -> Net-(Q1-Pad1)
- R7 pad 2: Net-(Q2-Pad2) -> Net-(Q2-Pad1)
- U1 pad 29: GND -> (no net)
Routing:
- net V_USB: track 171.0 -> 487.3 mm, vias 5 -> 39
- net GND: track 161.1 -> 457.9 mm, vias 4 -> 33
- net Net-(LED14-Pad4): track 60.3 -> 0.00 mm, vias 6 -> 0
- net Net-(LED15-Pad4): track 58.9 -> 0.00 mm, vias 6 -> 0
- net Net-(LED13-Pad4): track 58.9 -> 0.00 mm, vias 6 -> 0
- net Net-(LED16-Pad4): track 57.8 -> 0.00 mm, vias 6 -> 0
- net Net-(LED13-Pad3): track 54.0 -> 0.00 mm, vias 5 -> 0
- net Net-(LED15-Pad3): track 53.3 -> 0.00 mm, vias 5 -> 0
- net Net-(LED16-Pad3): track 53.2 -> 0.00 mm, vias 5 -> 0
- net Net-(LED14-Pad3): track 52.6 -> 0.00 mm, vias 5 -> 0
- net Net-(LED41-Pad4): track 31.5 -> 0.00 mm, vias 4 -> 0
- net Net-(LED41-Pad3): track 26.6 -> 0.00 mm, vias 3 -> 0
- net Net-(LED44-Pad4): track 24.6 -> 0.00 mm, vias 3 -> 0
- net Net-(LED42-Pad4): track 24.2 -> 0.00 mm, vias 3 -> 0
- net Net-(LED44-Pad3): track 19.5 -> 0.00 mm, vias 2 -> 0
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- added copper zone on B.Cu, net GND
- added copper zone on F.Cu, net V_USB
Other:
- board text added: "esp8266_apa102_bulb v4.1"
- board text removed: "esp8266_apa102_bulb v4.0"
