File: hardware/led_bulb.sch (KiCad schematic (older format))
At the start: 112 parts, among them P1 USB_OTG, P10 CONN_01X02, P11 CONN_01X02, P12 CONN_01X02, P13 CONN_01X02, P14 CONN_01X02, P15 CONN_01X02, P16 CONN_01X02, P17 CONN_01X02, P18 CONN_01X02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

Commit message: Changed U4/C7/C8/C10 footprint sizes
Changed lines of the file:
@@
 Wire Wire Line
 	7550 4600 7650 4600
-$Sheet
-S 2500 -850 850  850
-U 57994C96
-F0 "apa102" 60
-F1 "apa102.sch" 60
-$EndSheet
 $Comp
 L Q_NPN_BEC Q2
